File: PCB/ECEN2270-Final Project.brd (EAGLE design)
At the start: 54.6 x 39 mm, 41 parts, among them J1 USB_MINI-B_SMT, J2 POWER_JACK, Q1 310mA/60V/1.6Ω, Q2 2.5A/30V/105mΩ, U1 FT231XS, U2 LMV358, U3 ATMEGA328P_TQFP, U4 3.3V/150mA, Y2 16MHz

Commit message: Replaced Mini USB with Micro
Parts:
- J1: value USB_MINI-B_SMT -> (none); device SparkFun-Connectors:USB-MINIB -> SparkFun-Connectors:USB-B-MICRO-SMD
- moved J1 3.81 mm to (2.54, 21.6)
Connections:
- net GND: now also J1.SHIELD1, J1.SHIELD2, J1.SHIELD3; no longer J1.S1, J1.S2, J1.S3, J1.S4
Routing:
- net GND: track 215.9 -> 200.7 mm
- net N$2: track 18.6 -> 11.8 mm
- net N$4: track 24.3 -> 19.9 mm
- net N$1: track 7.20 -> 10.1 mm
